Commit message: robo atualizad

File: urdf/pioneer3dx.urdf (robot description, URDF)
Before this commit: robot pioneer3dx, 11 links, 10 joints
Links:
- added link brush; collision box size=0.12 1.45 0.15; visual box size=0.12 1.45 0.15
- added link brush_support; collision box size=0.15 1.5 0.02; visual box size=0.15 1.5 0.02
- added link handle; visual cylinder length=1 radius=0.025
Joints:
- added joint handle_to_brush_support: type fixed, parent handle, child brush_support, origin xyz=-0.70710678 0 -0.70710678 rpy=0 0 0
- added joint handle_to_robot: type continuous, parent top_plate, child handle, origin xyz=-0.2 0 0.05 rpy=0 0.78539816339 0, axis 0 1 0
- added joint suport_to_brush: type fixed, parent brush_support, child brush, origin xyz=0 0 0 rpy=0 0 0

Commit message: finalizacao do modelo do robo sem variaveis fisicas

File: urdf/pioneer3dx.urdf (robot description, URDF)
Before this commit: robot pioneer3dx, 14 links, 13 joints
Links:
- added link y_cilinder_joint; visual cylinder length=0.05 radius=0.025
- added link z_cilinder_joint; visual cylinder length=0.05 radius=0.025
Joints:
- added joint y_cilinder_joint_to_robot: type continuous, parent z_cilinder_joint, child y_cilinder_joint, origin xyz=0 0 0.025 rpy=0 0 0, axis 0 1 0
- added joint z_cilinder_joint_to_robot: type continuous, parent top_plate, child z_cilinder_joint, origin xyz=-0.2 0 0.025 rpy=0 0 0, axis 0 0 1
- joint handle_to_robot: axis 0 1 0 -> (none); origin xyz=-0.2 0 0.05 rpy=0 0.78539816339 0 -> xyz=0 0 0 rpy=0 0.78539816339 0; parent top_plate -> y_cilinder_joint; type continuous -> fixed
