Commit message: adicao de momentos de inercia porem necessario correcao de movimentos anomalos

File: tennis_bot/urdf/pioneer3dx.urdf (robot description, URDF)
Before this commit: robot pioneer3dx, 16 links, 15 joints
Links:
- link brush: mass None -> 1
- link brush_support: mass None -> 10
- link handle: mass None -> 1; geometry collision cylinder length=1 radius=0.025; visual cylinder length=1 radius=0.025
- link y_cilinder_joint: mass None -> 1; geometry collision cylinder length=0.05 radius=0.025; visual cylinder length=0.05 radius=0.025
- link z_cilinder_joint: mass None -> 1; geometry collision cylinder length=0.05 radius=0.025; visual cylinder length=0.05 radius=0.025

File: tennis_bot/urdf/pioneer3dx.xacro (robot description, xacro)
@@ -167,9 +167,4 @@
 	</material>
 	<link name="z_cilinder_joint">
-		<inertial>
-			<origin xyz="0 0 0" rpy="0 0 0"/>
-			<mass value="0.1"/>
-			<inertia ixx="0.0001" ixy="0.0" ixz="0.0" iyy="0.0001" iyz="0.0" izz="0.0001"/>
-		</inertial>
 		<visual>
 			<geometry>
@@ -178,11 +173,16 @@
 			<material name="pink"/>
 			<origin rpy="0 0 0" xyz="0 0 0"/>
-			<collision>
-				<geometry>
-					<cylinder length="0.05" radius="0.025"/>
-				</geometry>
-				<origin rpy="0 0 0" xyz="0 0 0"/>
-			</collision>
-		</visual>
+		</visual>
+		<collision>
+			<geometry>
+				<cylinder length="0.05" radius="0.025"/>
+			</geometry>
+			<origin rpy="0 0 0" xyz="0 0 0"/>
+		</collision>
+		<inertial>
+			<origin xyz="0 0 0" rpy="0 0 0"/>
+			<mass value="1"/>
+			<inertia ixx="0.000365" ixy="0.0" ixz="0.0" iyy="0.000365" iyz="0.0" izz="0.000313"/>
+		</inertial>
 	</link>
 	<gazebo reference="z_cilinder_joint">
@@ -202,11 +202,16 @@
 			<material name="pink"/>
 			<origin rpy="1.57079632679 0 0" xyz="0 0 0"/>
-			<collision>
-				<geometry>
-					<cylinder length="0.05" radius="0.025"/>
-				</geometry>
-				<origin rpy="1.57079632679 0 0" xyz="0 0 0"/>
-			</collision>
-		</visual>
+		</visual>
+		<collision>
+			<geometry>
+				<cylinder length="0.05" radius="0.025"/>
+			</geometry>
+			<origin rpy="1.57079632679 0 0" xyz="0 0 0"/>
+		</collision>
+		<inertial>
+			<origin xyz="0 0 0" rpy="0 0 0"/>
+			<mass value="1"/>
+			<inertia ixx="0.000365" ixy="0.0" ixz="0.0" iyy="0.000365" iyz="0.0" izz="0.000313"/>
+		</inertial>
 	</link>
 	<gazebo reference="y_cilinder_joint">
@@ -226,11 +231,16 @@
 			<material name="brown"/>
 			<origin rpy="0 0.78539816339 0" xyz="-0.35355339059 0 -0.35355339059"/>
-			<collision>
-				<geometry>
-					<cylinder length="1" radius="0.025"/>
-				</geometry>
-				<origin rpy="0 0.78539816339 0" xyz="-0.35355339059 0 -0.35355339059"/>
-			</collision>
-		</visual>
+		</visual>
+		<collision>
+			<geometry>
+				<cylinder length="1" radius="0.025"/>
+			</geometry>
+			<origin rpy="0 0.78539816339 0" xyz="-0.35355339059 0 -0.35355339059"/>
+		</collision>
+		<inertial>
+			<origin xyz="0 0 0" rpy="0 0 0"/>
+			<mass value="1"/>
+			<inertia ixx="0.083490" ixy="0.0" ixz="0.0" iyy="0.083490" iyz="0.0" izz="0.000313"/>
+		</inertial>
 	</link>
 	<gazebo reference="handle">
@@ -256,4 +266,9 @@
 			<origin rpy="0 0 0" xyz="0 0 0"/>
 		</collision>
+		<inertial>
+			<origin xyz="0 0 0" rpy="0 0 0"/>
+			<mass value="1"/>
+			<inertia ixx="0.1875330" ixy="0.0" ixz="0.0" iyy="0.0019080" iyz="0.0" izz="0.1893750"/>
+		</inertial>
 	</link>
 	<gazebo reference="brush_support">
@@ -279,4 +294,9 @@
 			<origin rpy="0 0 0" xyz="0 0 -0.075"/>
 		</collision>
+		<inertial>
+			<origin xyz="0 0 0" rpy="0 0 0"/>
+			<mass value="1"/>
+			<inertia ixx="0.177083" ixy="0.0" ixz="0.0" iyy="0.003075" iyz="0.0" izz="0.176408"/>
+		</inertial>
 	</link>
 	<gazebo reference="brush">
