Commit message: correcao de massas e inercias

File: tennis_bot/urdf/pioneer3dx.xacro (robot description, xacro)
@@ -174,14 +174,14 @@
 			<origin rpy="0 0 0" xyz="0 0 0"/>
 		</visual>
-		<collision>
+		<!-- <collision>
 			<geometry>
 				<cylinder length="0.05" radius="0.025"/>
 			</geometry>
 			<origin rpy="0 0 0" xyz="0 0 0"/>
-		</collision>
-		<inertial>
-			<origin xyz="0 0 0" rpy="0 0 0"/>
-			<mass value="1"/>
-			<inertia ixx="0.000365" ixy="0.0" ixz="0.0" iyy="0.000365" iyz="0.0" izz="0.000313"/>
+		</collision> -->
+		<inertial>
+			<origin xyz="0 0 0" rpy="0 0 0"/>
+			<mass value="0.05"/>
+			<inertia ixx="0.00001823" ixy="0.0" ixz="0.0" iyy="0.00001823" iyz="0.0" izz="0.00001563"/>
 		</inertial>
 	</link>
@@ -203,14 +203,14 @@
 			<origin rpy="1.57079632679 0 0" xyz="0 0 0"/>
 		</visual>
-		<collision>
+		<!-- <collision>
 			<geometry>
 				<cylinder length="0.05" radius="0.025"/>
 			</geometry>
 			<origin rpy="1.57079632679 0 0" xyz="0 0 0"/>
-		</collision>
-		<inertial>
-			<origin xyz="0 0 0" rpy="0 0 0"/>
-			<mass value="1"/>
-			<inertia ixx="0.000365" ixy="0.0" ixz="0.0" iyy="0.000365" iyz="0.0" izz="0.000313"/>
+		</collision> -->
+		<inertial>
+			<origin xyz="0 0 0" rpy="0 0 0"/>
+			<mass value="0.05"/>
+			<inertia ixx="0.00001823" ixy="0.0" ixz="0.0" iyy="0.00001823" iyz="0.0" izz="0.00001563"/>
 		</inertial>
 	</link>
@@ -240,6 +240,6 @@
 		<inertial>
 			<origin xyz="0 0 0" rpy="0 0 0"/>
-			<mass value="1"/>
-			<inertia ixx="0.083490" ixy="0.0" ixz="0.0" iyy="0.083490" iyz="0.0" izz="0.000313"/>
+			<mass value="0.3"/>
+			<inertia ixx="0.02504687" ixy="0.0" ixz="0.0" iyy="0.02504687" iyz="0.0" izz="0.00009375"/>
 		</inertial>
 	</link>
@@ -268,6 +268,6 @@
 		<inertial>
 			<origin xyz="0 0 0" rpy="0 0 0"/>
-			<mass value="1"/>
-			<inertia ixx="0.1875330" ixy="0.0" ixz="0.0" iyy="0.0019080" iyz="0.0" izz="0.1893750"/>
+			<mass value="0.3"/>
+			<inertia ixx="0.05626" ixy="0.0" ixz="0.0" iyy="0.0005725" iyz="0.0" izz="0.0568125"/>
 		</inertial>
 	</link>
@@ -296,10 +296,14 @@
 		<inertial>
 			<origin xyz="0 0 0" rpy="0 0 0"/>
-			<mass value="1"/>
-			<inertia ixx="0.177083" ixy="0.0" ixz="0.0" iyy="0.003075" iyz="0.0" izz="0.176408"/>
+			<mass value="0.2"/>
+			<inertia ixx="0.03541667" ixy="0.0" ixz="0.0" iyy="0.000615" iyz="0.0" izz="0.03528167"/>
 		</inertial>
 	</link>
 	<gazebo reference="brush">
 		<material>Gazebo/Black</material>
+		<mu1>2</mu1>
+		<mu2>2</mu2>
+		<kp>10000.0</kp>
+		<kd>10.0</kd>
 	</gazebo>
 	<joint name="suport_to_brush" type="fixed">

Commit message: adicao da quadra aos launchs, ainda sao necessarios ajustes nas posicoes de spawn de cada robo

File: tennis_bot/urdf/pioneer3dx.xacro (robot description, xacro)
@@ -268,6 +268,6 @@
 		<inertial>
 			<origin xyz="0 0 0" rpy="0 0 0"/>
-			<mass value="0.3"/>
-			<inertia ixx="0.05626" ixy="0.0" ixz="0.0" iyy="0.0005725" iyz="0.0" izz="0.0568125"/>
+			<mass value="0.8"/>
+			<inertia ixx="0.15002667" ixy="0.0" ixz="0.0" iyy="0.00152667" iyz="0.0" izz="0.1515"/>
 		</inertial>
 	</link>
@@ -283,25 +283,25 @@
 		<visual>
 			<geometry>
-				<box size="0.12 1.45 0.15"/>
-			</geometry>
-			<origin rpy="0 0 0" xyz="0 0 -0.075"/>
+				<box size="0.12 1.45 0.09"/>
+			</geometry>
+			<origin rpy="0 0 0" xyz="0 0 -0.045"/>
 			<material name="green"/>
 		</visual>
 		<collision>
 			<geometry>
-				<box size="0.12 1.45 0.15"/>
-			</geometry>
-			<origin rpy="0 0 0" xyz="0 0 -0.075"/>
+				<box size="0.12 1.45 0.09"/>
+			</geometry>
+			<origin rpy="0 0 0" xyz="0 0 -0.045"/>
 		</collision>
 		<inertial>
 			<origin xyz="0 0 0" rpy="0 0 0"/>
 			<mass value="0.2"/>
-			<inertia ixx="0.03541667" ixy="0.0" ixz="0.0" iyy="0.000615" iyz="0.0" izz="0.03528167"/>
+			<inertia ixx="0.03517667" ixy="0.0" ixz="0.0" iyy="0.000375" iyz="0.0" izz="0.03528167"/>
 		</inertial>
 	</link>
 	<gazebo reference="brush">
 		<material>Gazebo/Black</material>
-		<mu1>2</mu1>
-		<mu2>2</mu2>
+		<mu1>1</mu1>
+		<mu2>1.0</mu2>
 		<kp>10000.0</kp>
 		<kd>10.0</kd>
